Commit message: change ur base frame as 0, not finish

File: Meshes/ur10_origin.urdf (robot description, URDF)
Before this commit: robot ur10, 9 links, 8 joints
Joints:
- joint world_joint: origin xyz=0.0 0.0 1.0 rpy=0.0 0.0 0.0 -> xyz=0.0 0.0 0.0 rpy=0.0 0.0 0.0

File: Meshes/ur10_tactile.urdf (robot description, URDF)
Before this commit: robot ur10, 10 links, 9 joints
Joints:
- joint digit_joint: origin xyz=0.1 0 0 rpy=0 -1.570796325 0 -> xyz=0.1 0 0 rpy=0 1.570796325 3.141592654
- joint world_joint: origin xyz=0.0 0.0 1.0 rpy=0.0 0.0 0.0 -> xyz=0.0 0.0 0.0 rpy=0.0 0.0 0.0
