Commit message: add contact test and figure process

File: Meshes/ur10_tactile.urdf (robot description, URDF)
Before this commit: robot ur10, 9 links, 8 joints
Links:
- added link digit_link, mass 0.1; collision mesh filename=digit.STL; visual mesh filename=digit.STL
Joints:
- added joint digit_joint: type fixed, parent ee_link, child digit_link, origin xyz=0.1 0 0 rpy=0 -1.570796325 0

Commit message: remove self collision

File: Meshes/ur10_tactile.urdf (robot description, URDF)
Before this commit: robot ur10, 10 links, 9 joints
Links:
- link base_link: geometry visual mesh filename=package://ur_description/meshes/ur10/visual/Base.dae
- link ee_link: geometry visual box size=0.05 0.05 0.05
- link forearm_link: geometry visual mesh filename=package://ur_description/meshes/ur10/visual/Forearm.dae
- link shoulder_link: geometry visual mesh filename=package://ur_description/meshes/ur10/visual/Shoulder.dae
- link upper_arm_link: geometry visual mesh filename=package://ur_description/meshes/ur10/visual/UpperArm.dae
- link wrist_1_link: geometry visual mesh filename=package://ur_description/meshes/ur10/visual/Wrist1.dae
- link wrist_2_link: geometry visual mesh filename=package://ur_description/meshes/ur10/visual/Wrist2.dae
- link wrist_3_link: geometry visual mesh filename=package://ur_description/meshes/ur10/visual/Wrist3.dae
